File: main/pcb_challenge_final.kicad_sch (KiCad schematic)
At the start: 164 parts, among them J4 Conn_01x04_Pin, J5 Conn_01x04_Pin, Q15 Q_Dual_NPN_PNP_B1E2B2C2E1C1, Q16 Q_Dual_NPN_PNP_B1E2B2C2E1C1, Q17 Q_Dual_NPN_PNP_B1E2B2C2E1C1, Q18 Q_Dual_NPN_PNP_B1E2B2C2E1C1, Q19 Q_Dual_NPN_PNP_B1E2B2C2E1C1, Q20 Q_Dual_NPN_PNP_B1E2B2C2E1C1, Q21 Q_Dual_NPN_PNP_B1E2B2C2E1C1, Q22 Q_Dual_NPN_PNP_B1E2B2C2E1C1, Q23 Q_Dual_NPN_PNP_B1E2B2C2E1C1, Q24 Q_Dual_NPN_PNP_B1E2B2C2E1C1, Q25 Q_Dual_NPN_PNP_B1E2B2C2E1C1, Q26 Q_Dual_NPN_PNP_B1E2B2C2E1C1, Q27 Q_Dual_NPN_PNP_B1E2B2C2E1C1, Q28 Q_Dual_NPN_PNP_B1E2B2C2E1C1, Q29 Q_Dual_NPN_PNP_B1E2B2C2E1C1, SW1 SW_Push, SW2 SW_MEC_5G, SW3 SW_Push, U1 74AUP1G80, U10 NMUX1308BQ, U11 NMUX1308BQ, U12 NMUX1308BQ, U13 NMUX1308BQ, U14 NMUX1308BQ, U15 NMUX1308BQ, U16 NMUX1308BQ, U17 74AUP1G80, U18 74AHC1G86, U19 74AUP1G80, U20 74AUP1G80, U21 74LV1T08GV, U22 CD74HC283M96, U23 74LV1T08GV, U24 74LVC1GU04DRL, U25 ESP32-S3-MINI-1, U26 74LVC1GU04DRL, U27 74LV1T08GV, U28 CD74HC283M96, U29 NMUX1308BQ, U3 74AHC1G86, U30 NMUX1308BQ, U31 NMUX1308BQ, U32 NMUX1308BQ, U33 74AUP1G80, U34 74AUP1G80, U35 NMUX1308BQ, U36 NMUX1308BQ, U37 74AUP1G80, U38 74AUP1G80, U39 NMUX1308BQ, U4 74AUP1G80, U40 NMUX1308BQ, U41 NMUX1308BQ, U42 NMUX1308BQ, U43 NMUX1308BQ, U44 NMUX1308BQ, U45 74AUP1G80, U46 74AUP1G80, U47 74AUP1G80, U48 74AUP1G80, U49 74AUP1G80, U5 74AUP1G80, U50 74AUP1G80, U51 74LV1T08GV, U52 74AHC1G86, U53 74LVC1GU04DRL, U54 74LVC1GU04DRL, U55 74AHC1G86, U56 74AHC1G86, U57 74LVC1GU04DRL, U58 74LVC1GU04DRL, U59 74LV1T08GV, U6 74AUP1G80, U60 74AHC1G86, U61 74LVC1GU04DRL, U62 74LV1T08GV, U63 74LV1T08GV, U64 NMUX1308BQ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

Commit message: PCB Challenge 2026 submission - Mickey
Connections:
- net EN is gone; now on net en: Y2.1 (INH)
Other:
- moved on the sheet: SW2
Changed lines of the file:
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@@
 	(wire
 		(pts
-			(xy 83.82 40.64) (xy 93.98 40.64)
+			(xy 82.55 40.64) (xy 93.98 40.64)
 		)
 		(stroke
@@
 	(wire
 		(pts
+			(xy 92.71 30.48) (xy 93.98 30.48)
+		)
+		(stroke
+			(width 0)
+			(type default)
+		)
+	)
+	(wire
+		(pts
 			(xy 275.59 384.81) (xy 257.81 384.81)
 		)
@@
 	(wire
 		(pts
-			(xy 83.82 30.48) (xy 83.82 40.64)
+			(xy 82.55 30.48) (xy 82.55 40.64)
 		)
 		(stroke
@@
 	(wire
 		(pts
-			(xy 93.98 30.48) (xy 95.25 30.48)
+			(xy 93.98 30.48) (xy 97.79 30.48)
 		)
 		(stroke
@@
 		)
 	)
-	(global_label "EN"
+	(global_label "en"
 		(shape input)
 		(at 36.83 71.12 180)
@@
 		)
 		(property "Intersheetrefs" "${INTERSHEET_REFS}"
-			(at 31.3653 71.12 0)
+			(at 31.6072 71.12 0)
 			(hide yes)
 			(show_name no)
@@
 	(global_label "NRST"
 		(shape input)
-		(at 95.25 30.48 0)
+		(at 97.79 30.48 0)
 		(fields_autoplaced yes)
 		(effects
@@
 		)
 		(property "Intersheetrefs" "${INTERSHEET_REFS}"
-			(at 103.0128 30.48 0)
+			(at 105.5528 30.48 0)
 			(hide yes)
 			(show_name no)
@@
 	(symbol
 		(lib_id "Switch:SW_MEC_5G")
-		(at 88.9 30.48 0)
+		(at 87.63 30.48 0)
 		(unit 1)
 		(body_style 1)
@@
 		(dnp no)
 		(property "Reference" "SW2"
-			(at 88.9 26.162 0)
+			(at 87.63 26.162 0)
 			(show_name no)
 			(do_not_autoplace no)
@@
 		)
 		(property "Value" "SW_MEC_5G"
-			(at 88.9 25.4 0)
+			(at 87.63 25.4 0)
 			(hide yes)
 			(show_name no)
@@
 		)
 		(property "Footprint" "Button_Switch_SMD:SW_SPST_CK_RS282G05A3"
-			(at 88.9 25.4 0)
+			(at 87.63 25.4 0)
 			(hide yes)
 			(show_name no)
@@
 		)
 		(property "Datasheet" "https://www.apem.com/medias/download/MEC_switches_serie_MULTIMEC5G.pdf"
-			(at 88.9 25.4 0)
+			(at 87.63 25.4 0)
 			(hide yes)
 			(show_name no)
@@
 		)
 		(property "Description" "MEC 5G single pole normally-open tactile switch"
-			(at 88.9 30.48 0)
+			(at 87.63 30.48 0)
 			(hide yes)
 			(show_name no)
